File: LO_PCB/LO_PCB.kicad_sch (KiCad schematic)
At the start: 116 parts, among them J1 OSCinP, J2 OSCinM, J3 PWR, J4 Conn_01x08, J5 LO_OUT_A, J6 LO_OUT_A, Q1 AO3401A, U1 LMX2582RHAR, U2 TPS7A9101DSKT, U3 PE42424A-Z, U4 PE42424A-Z, U5 PE42424A-Z, U6 PE42424A-Z

Commit message: schematic finished for LO pcb
Parts:
- removed C50, C51, C60, C61: 100pF, symbol Device:C
- removed C52, C59: 10nF, symbol Device:C
- removed C53, C57: 3.6pF, symbol Device:C
- removed C54, C58: 1.2pF, symbol Device:C
- removed C55: 6.2pF, symbol Device:C
- removed C56: 2pF, symbol Device:C
- removed J2: OSCinM, symbol Connector:Conn_Coaxial
- removed J6: LO_OUT_A, symbol Connector:Conn_Coaxial
- removed R4: 18, symbol Device:R
- removed U6: PE42424A-Z, Snapeda:DFN6_1P5X1P5-0P5_PSM, symbol Snapeda:PE42424A-Z
- added C19, C21: 3.9pF, Capacitor_SMD:C_0402_1005Metric, symbol Device:C
- added C20: 6.8pF, Capacitor_SMD:C_0402_1005Metric, symbol Device:C
- added C22, C23, C24, C27: 100pF, Capacitor_SMD:C_0402_1005Metric, symbol Device:C
- added C25, C26: 10nF, Capacitor_SMD:C_0402_1005Metric, symbol Device:C
- added C32, C34: 1.3pF, Capacitor_SMD:C_0402_1005Metric, symbol Device:C
- added C33: 2.2pF, Capacitor_SMD:C_0402_1005Metric, symbol Device:C
- added C43, C45, C48: 10uF, Capacitor_SMD:C_0603_1608Metric, symbol Device:C
- added J3: LO_OUT_B, Snapeda:J_Wurth_WR-SMA_60312202114513, symbol Connector:Conn_Coaxial
- added R21, R34, R36: 10k, Resistor_SMD:R_0603_1608Metric, symbol Device:R
- added U4: PE42424A-Z, Snapeda:DFN6_1P5X1P5-0P5_PSM, symbol Snapeda:PE42424A-Z
- C1: renamed from C42; value 3.6pF -> 3.9pF; footprint (none) -> Capacitor_SMD:C_0402_1005Metric; Dielectric (none) -> C0G; Tolerance (none) -> +/-0.1pF; Voltage (none) -> 50V
- C10: renamed from C41; footprint (none) -> Capacitor_SMD:C_0402_1005Metric; Dielectric (none) -> C0G; Tolerance (none) -> +/-5%; Voltage (none) -> 50V
- C11: renamed from C40; footprint (none) -> Capacitor_SMD:C_0402_1005Metric; Dielectric (none) -> C0G; Tolerance (none) -> +/-5%; Voltage (none) -> 50V
- C12: renamed from C39; footprint (none) -> Capacitor_SMD:C_0402_1005Metric; Dielectric (none) -> X7R; Tolerance (none) -> +/-10%; Voltage (none) -> 25V
- C13: renamed from C44; footprint (none) -> Capacitor_SMD:C_0402_1005Metric; Dielectric (none) -> X7R; Tolerance (none) -> +/-10%; Voltage (none) -> 25V
- C14: renamed from C43; footprint (none) -> Capacitor_SMD:C_0402_1005Metric; Dielectric (none) -> C0G; Tolerance (none) -> +/-5%; Voltage (none) -> 50V
- C15: renamed from C12; footprint (none) -> Capacitor_SMD:C_0603_1608Metric; Dielectric (none) -> X7R; Tolerance (none) -> +/-10%; Voltage (none) -> 25V
- C16: renamed from C47; value 1.2pF -> 1.3pF; footprint (none) -> Capacitor_SMD:C_0402_1005Metric; Dielectric (none) -> C0G; Tolerance (none) -> +/-0.1pF; Voltage (none) -> 50V
- C17: renamed from C48; value 2pF -> 2.2pF; footprint (none) -> Capacitor_SMD:C_0402_1005Metric; Dielectric (none) -> C0G; Tolerance (none) -> +/-0.1pF; Voltage (none) -> 50V
- C18: renamed from C49; value 1.2pF -> 1.3pF; footprint (none) -> Capacitor_SMD:C_0402_1005Metric; Dielectric (none) -> C0G; Tolerance (none) -> +/-0.1pF; Voltage (none) -> 50V
- C2: renamed from C45; value 6.2pF -> 6.8pF; footprint (none) -> Capacitor_SMD:C_0402_1005Metric; Dielectric (none) -> C0G; Tolerance (none) -> +/-0.1pF; Voltage (none) -> 50V
- C28: renamed from C20; footprint (none) -> Capacitor_SMD:C_0603_1608Metric; Dielectric (none) -> X7R; Tolerance (none) -> +/-10%; Voltage (none) -> 25V
- C29: renamed from C21; footprint (none) -> Capacitor_SMD:C_0603_1608Metric; Dielectric (none) -> X5R; Tolerance (none) -> +/-20%; Voltage (none) -> 16V
- C3: renamed from C46; value 3.6pF -> 3.9pF; footprint (none) -> Capacitor_SMD:C_0402_1005Metric; Dielectric (none) -> C0G; Tolerance (none) -> +/-0.1pF; Voltage (none) -> 50V
- C30: renamed from C24; footprint (none) -> Capacitor_SMD:C_0603_1608Metric; Dielectric (none) -> X7R; Tolerance (none) -> +/-10%; Voltage (none) -> 25V
- C31: renamed from C25; footprint (none) -> Capacitor_SMD:C_0603_1608Metric; Dielectric (none) -> X5R; Tolerance (none) -> +/-20%; Voltage (none) -> 16V
- C35: renamed from C22; footprint (none) -> Capacitor_SMD:C_0603_1608Metric; Dielectric (none) -> X7R; Tolerance (none) -> +/-10%; Voltage (none) -> 25V
- C36: renamed from C23; footprint (none) -> Capacitor_SMD:C_0603_1608Metric; Dielectric (none) -> X5R; Tolerance (none) -> +/-20%; Voltage (none) -> 16V
- C37: renamed from C26; footprint (none) -> Capacitor_SMD:C_0603_1608Metric; Dielectric (none) -> X7R; Tolerance (none) -> +/-10%; Voltage (none) -> 25V
- C38: renamed from C27; footprint (none) -> Capacitor_SMD:C_0603_1608Metric; Dielectric (none) -> X5R; Tolerance (none) -> +/-20%; Voltage (none) -> 16V
- C39: renamed from C33; footprint (none) -> Capacitor_SMD:C_0402_1005Metric; Dielectric (none) -> X7R; Tolerance (none) -> +/-10%; Voltage (none) -> 25V
- C4: renamed from C14; footprint (none) -> Capacitor_SMD:C_0603_1608Metric; Dielectric (none) -> X7R; Tolerance (none) -> +/-10%; Voltage (none) -> 25V
- C40: renamed from C37; footprint (none) -> Capacitor_SMD:C_0402_1005Metric; Dielectric (none) -> X7R; Tolerance (none) -> +/-10%; Voltage (none) -> 25V
- C41: renamed from C18; footprint (none) -> Capacitor_SMD:C_0402_1005Metric; Dielectric (none) -> C0G; Tolerance (none) -> +/-5%; Voltage (none) -> 50V
- C42: renamed from C28; footprint (none) -> Capacitor_SMD:C_0402_1005Metric; Dielectric (none) -> X7R; Tolerance (none) -> +/-10%; Voltage (none) -> 25V
- C44: renamed from C29; footprint (none) -> Capacitor_SMD:C_0402_1005Metric; Dielectric (none) -> X7R; Tolerance (none) -> +/-10%; Voltage (none) -> 25V
- C46: renamed from C30; footprint (none) -> Capacitor_SMD:C_0402_1005Metric; Dielectric (none) -> X7R; Tolerance (none) -> +/-10%; Voltage (none) -> 25V
- C47: renamed from C31; footprint (none) -> Capacitor_SMD:C_0402_1005Metric; Dielectric (none) -> X7R; Tolerance (none) -> +/-10%; Voltage (none) -> 25V
- C49: renamed from C32; footprint (none) -> Capacitor_SMD:C_0402_1005Metric; Dielectric (none) -> X7R; Tolerance (none) -> +/-10%; Voltage (none) -> 25V
- C5: renamed from C11; footprint (none) -> Capacitor_SMD:C_0603_1608Metric; Dielectric (none) -> X5R; Tolerance (none) -> +/-20%; Voltage (none) -> 16V
- C50: renamed from C16; footprint (none) -> Capacitor_SMD:C_0402_1005Metric; Dielectric (none) -> C0G; Tolerance (none) -> +/-5%; Voltage (none) -> 50V
- C51: renamed from C17; footprint (none) -> Capacitor_SMD:C_0402_1005Metric; Dielectric (none) -> C0G; Tolerance (none) -> +/-5%; Voltage (none) -> 50V
- C52: renamed from C4; footprint (none) -> Capacitor_SMD:C_0603_1608Metric; Dielectric (none) -> X7R; Tolerance (none) -> +/-10%; Voltage (none) -> 25V
- C53: renamed from C36; footprint (none) -> Capacitor_SMD:C_0603_1608Metric; Dielectric (none) -> C0G; Tolerance (none) -> +/-5%; Voltage (none) -> 50V
- C54: renamed from C35; footprint (none) -> Capacitor_SMD:C_0805_2012Metric; Dielectric (none) -> X7R; Tolerance (none) -> +/-10%; Voltage (none) -> 25V
- C55: renamed from C5; footprint (none) -> Capacitor_SMD:C_0603_1608Metric; Dielectric (none) -> X5R; Tolerance (none) -> +/-20%; Voltage (none) -> 16V
- C56: renamed from C34; footprint (none) -> Capacitor_SMD:C_0603_1608Metric; Dielectric (none) -> C0G; Tolerance (none) -> +/-5%; Voltage (none) -> 50V
- C57: renamed from C6; footprint (none) -> Capacitor_SMD:C_0603_1608Metric; Dielectric (none) -> X7R; Tolerance (none) -> +/-10%; Voltage (none) -> 25V
- C58: renamed from C7; footprint (none) -> Capacitor_SMD:C_0603_1608Metric; Dielectric (none) -> X5R; Tolerance (none) -> +/-20%; Voltage (none) -> 16V
- C59: renamed from C8; footprint (none) -> Capacitor_SMD:C_0603_1608Metric; Dielectric (none) -> X5R; Tolerance (none) -> +/-20%; Voltage (none) -> 16V
- C6: renamed from C19; footprint (none) -> Capacitor_SMD:C_0603_1608Metric; Dielectric (none) -> X7R; Tolerance (none) -> +/-10%; Voltage (none) -> 25V
- C60: renamed from C1; footprint (none) -> Capacitor_SMD:C_0603_1608Metric; Dielectric (none) -> X7R; Tolerance (none) -> +/-10%; Voltage (none) -> 25V
- C61: renamed from C9; footprint (none) -> Capacitor_SMD:C_0603_1608Metric; Dielectric (none) -> X7R; Tolerance (none) -> +/-10%; Voltage (none) -> 25V
- C62: renamed from C10; footprint (none) -> Capacitor_SMD:C_0603_1608Metric; Dielectric (none) -> X5R; Tolerance (none) -> +/-20%; Voltage (none) -> 16V
- C63: renamed from C2; footprint (none) -> Capacitor_SMD:C_0402_1005Metric; Dielectric (none) -> X7R; Tolerance (none) -> +/-10%; Voltage (none) -> 25V
- C64: renamed from C3; footprint (none) -> Capacitor_SMD:C_0402_1005Metric; Dielectric (none) -> X7R; Tolerance (none) -> +/-10%; Voltage (none) -> 25V
- C7: renamed from C13; footprint (none) -> Capacitor_SMD:C_0603_1608Metric; Dielectric (none) -> X5R; Tolerance (none) -> +/-20%; Voltage (none) -> 16V
- C8: renamed from C15; footprint (none) -> Capacitor_SMD:C_0603_1608Metric; Dielectric (none) -> X7R; Tolerance (none) -> +/-10%; Voltage (none) -> 25V
- C9: renamed from C38; footprint (none) -> Capacitor_SMD:C_0402_1005Metric; Dielectric (none) -> C0G; Tolerance (none) -> +/-5%; Voltage (none) -> 50V
- J2: renamed from J5; footprint (none) -> Snapeda:J_Wurth_WR-SMA_60312202114513
- J4: renamed from J1; footprint (none) -> Snapeda:J_Wurth_WR-SMA_60312202114513
- J6: renamed from J4; footprint (none) -> Connector_PinHeader_2.54mm:PinHeader_1x08_P2.54mm_Vertical
- L1, L2, L5: value 10nH -> 11nH; footprint (none) -> Inductor_SMD:L_0402_1005Metric; Tolerance (none) -> +/-5%
- L3, L4, L8: value 3.6nH -> 3.9nH; footprint (none) -> Inductor_SMD:L_0402_1005Metric; Tolerance (none) -> +/-5%
- L6: value 3.6nH -> 11nH; footprint (none) -> Inductor_SMD:L_0402_1005Metric; Tolerance (none) -> +/-5%
- L7: value 10nH -> 3.9nH; footprint (none) -> Inductor_SMD:L_0402_1005Metric; Tolerance (none) -> +/-5%
- R1: renamed from R9; footprint (none) -> Resistor_SMD:R_0603_1608Metric; Tolerance (none) -> +/-1%
- R10: renamed from R25; footprint (none) -> Resistor_SMD:R_0402_1005Metric; Tolerance (none) -> +/-5%
- R11: renamed from R26; footprint (none) -> Resistor_SMD:R_0402_1005Metric; Tolerance (none) -> +/-5%
- R12: renamed from R33; footprint (none) -> Resistor_SMD:R_0402_1005Metric; Tolerance (none) -> +/-1%
- R13: renamed from R32; footprint (none) -> Resistor_SMD:R_0402_1005Metric; Tolerance (none) -> +/-1%
- R14: renamed from R35; footprint (none) -> Resistor_SMD:R_0402_1005Metric; Tolerance (none) -> +/-1%
- R15: renamed from R34; footprint (none) -> Resistor_SMD:R_0402_1005Metric; Tolerance (none) -> +/-1%
- R16: renamed from R37; footprint (none) -> Resistor_SMD:R_0402_1005Metric; Tolerance (none) -> +/-1%
- R17: renamed from R36; footprint (none) -> Resistor_SMD:R_0402_1005Metric; Tolerance (none) -> +/-1%
- R18: renamed from R28; footprint (none) -> Resistor_SMD:R_0603_1608Metric; Tolerance (none) -> +/-1%
- R19: renamed from R20; footprint (none) -> Resistor_SMD:R_0603_1608Metric; Tolerance (none) -> +/-5%
- R2: renamed from R13; footprint (none) -> Resistor_SMD:R_0603_1608Metric; Tolerance (none) -> +/-5%
- R20: renamed from R27; footprint (none) -> Resistor_SMD:R_0603_1608Metric; Tolerance (none) -> +/-1%
- R22: renamed from R1; footprint (none) -> Resistor_SMD:R_0603_1608Metric; Tolerance (none) -> +/-5%
- R23: renamed from R2; footprint (none) -> Resistor_SMD:R_0402_1005Metric; Tolerance (none) -> +/-5%
- R24: renamed from R3; footprint (none) -> Resistor_SMD:R_0402_1005Metric; Tolerance (none) -> +/-5%
- R25: renamed from R7; footprint (none) -> Resistor_SMD:R_0402_1005Metric; Tolerance (none) -> +/-5%
- R27: renamed from R8; footprint (none) -> Resistor_SMD:R_0402_1005Metric; Tolerance (none) -> +/-5%
- R28: renamed from R5; footprint (none) -> Resistor_SMD:R_0402_1005Metric; Tolerance (none) -> +/-5%
- R29: renamed from R6; footprint (none) -> Resistor_SMD:R_0402_1005Metric; Tolerance (none) -> +/-5%
- R3: renamed from R10; footprint (none) -> Resistor_SMD:R_0603_1608Metric; Tolerance (none) -> +/-1%
- R30: renamed from R11; footprint (none) -> Resistor_SMD:R_0603_1608Metric; Tolerance (none) -> +/-5%
- R31: renamed from R12; footprint (none) -> Resistor_SMD:R_0603_1608Metric; Tolerance (none) -> +/-5%
- R32: renamed from R17; footprint (none) -> Resistor_SMD:R_0603_1608Metric; Tolerance (none) -> +/-5%
- R33: renamed from R18; footprint (none) -> Resistor_SMD:R_0603_1608Metric; Tolerance (none) -> +/-5%
- R35: renamed from R19; footprint (none) -> Resistor_SMD:R_0603_1608Metric; Tolerance (none) -> +/-5%
- R4: renamed from R30; footprint (none) -> Resistor_SMD:R_0603_1608Metric; Tolerance (none) -> +/-5%
- R5: renamed from R29; footprint (none) -> Resistor_SMD:R_0603_1608Metric; Tolerance (none) -> +/-5%
- R6: renamed from R21; footprint (none) -> Resistor_SMD:R_0402_1005Metric; Tolerance (none) -> +/-5%
- R7: renamed from R22; footprint (none) -> Resistor_SMD:R_0402_1005Metric; Tolerance (none) -> +/-5%
- R8: renamed from R23; footprint (none) -> Resistor_SMD:R_0402_1005Metric; Tolerance (none) -> +/-5%
- R9: renamed from R24; footprint (none) -> Resistor_SMD:R_0402_1005Metric; Tolerance (none) -> +/-5%
- renumbered J3 to J1, U3 to U1, U4 to U2, U2 to U3, U1 to U6
Connections:
- net PF_FIL_SW_IN is gone; now on net RF_FIL_SW_IN: J6.3 (Pin_3)
- net PF_FIL_SW_OUT is gone; now on net RF_FIL_SW_OUT: J6.2 (Pin_2)
- net GND: now also C19.2, C20.2, C21.2, C24.1, C25.1, C26.1, C27.1, C32.2, C33.2, C34.2, C43.2, C45.2, C48.2, J3.2 (Ext), R36.2, U4.5 (GND), U4.7 (EPAD); no longer J6.8 (Pin_8)
- net RFOUT_B: now also C22.1
- net RF_FIL_SW_IN: now also R34.2, U4.1 (V1); no longer U5.1 (V1)
- net RF_FIL_SW_OUT: now also U5.1 (V1), R36.1
- net VCC: now also R21.1, R34.1
- net VccRF: now also C24.2, C25.2, C26.2, C27.2, U4.3 (VDD)
- net at C44.1, R7.2, U6.26 (VCCVCO2): now also C45.1
- net at R32.2: now also J6.7 (Pin_7); no longer J6.6 (Pin_6)
- net at C42.1, R6.2, U6.37 (VCCVCO): now also C43.1
- net at R31.2: now also J6.8 (Pin_8); no longer J6.7 (Pin_7)
- net at C47.1, R9.2, U6.15 (VCCMASH): now also C48.1
- net at L6.2: now also U5.4 (RF2), C21.1; no longer L8.1
- net at L7.2: now also L8.1, C33.1
- net at R35.2: now also J6.5 (Pin_5); no longer J6.4 (Pin_4)
- net at R33.2: now also J6.6 (Pin_6); no longer J6.5 (Pin_5)
- net at L6.1: now also L5.2, C20.1; no longer U5.6 (RF2)
- net INT_OSC_ENABLE: now reaches XTAL1.1 (E/D)
- net INT_OSC_ENABLE: now also J6.4 (Pin_4), R21.2
- net at C18.1, L4.2: now also U2.6 (RF1); no longer U2.4 (RF2)
- net at L8.2: now also U5.6 (RF1), C34.1
- net at C3.1, L2.2: now also U2.4 (RF2); no longer U2.6 (RF1)
- net at L7.1: now also C32.1, U4.4 (RF2); no longer L5.2
- net at U5.2 (RFC): now also C23.1
- net at L5.1: now also C19.1, U4.6 (RF1); no longer U5.4 (RF1)
- new net: C23.2, J3.1 (In)
- new net: C22.2, U4.2 (RFC)
- no-connect marks 6 -> 5
Other:
- note added: "External Input Reference SMA, Single Ended"
- note removed: "External Input Reference SMA"
- moved on the sheet: C15, C28, C29, C30, C31, C35, C36, C37, C38, C39, C4, C40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

Commit message: started on layout
Parts:
- removed C43, C45, C48: 10uF, Capacitor_SMD:C_0603_1608Metric, symbol Device:C
- added C41: 10nF, Capacitor_SMD:C_0402_1005Metric, symbol Device:C
- added C42: 100pF, Capacitor_SMD:C_0402_1005Metric, symbol Device:C
- renumbered C40 to C39, C41 to C40, C39 to C43, C42 to C44, C44 to C45, C49 to C48, C50 to C49, C51 to C50, C52 to C51, C53 to C52, C54 to C53, C55 to C54, C56 to C55, C57 to C56, C58 to C57, C59 to C58, C60 to C59, C61 to C60, C62 to C61, C63 to C62, C64 to C63, J6 to J5, R27 to R26, R28 to R27, R29 to R28, R30 to R29, R31 to R30, R32 to R31, R33 to R32, R34 to R33, R35 to R34, R36 to R35
Connections:
- net GND: now also C41.1, C42.1
- net VccRF: now also C41.2, C42.2
- net RF_FIL_SW_IN renamed FIL_SW_IN
- net RF_FIL_SW_OUT renamed FIL_SW_OUT
Other:
- moved on the sheet: C28, C29, C30, C31, C35, C36, C37, C38, C39, C40, C44, C45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

Commit message: initial placement done, todo: CPWG and all the other routing
Parts:
- removed C11, C14, C22, C24, C27: 100pF, Capacitor_SMD:C_0402_1005Metric, symbol Device:C
- removed C12, C13, C25, C26: 10nF, Capacitor_SMD:C_0402_1005Metric, symbol Device:C
- removed C16, C18, C32, C34: 1.3pF, Capacitor_SMD:C_0402_1005Metric, symbol Device:C
- removed C17, C33: 2.2pF, Capacitor_SMD:C_0402_1005Metric, symbol Device:C
- removed C19, C21: 3.9pF, Capacitor_SMD:C_0402_1005Metric, symbol Device:C
- removed C20: 6.8pF, Capacitor_SMD:C_0402_1005Metric, symbol Device:C
- removed L3, L4, L7, L8: 3.9nH, Inductor_SMD:L_0402_1005Metric, symbol Device:L
- removed L5, L6: 11nH, Inductor_SMD:L_0402_1005Metric, symbol Device:L
- removed R16: 49.9, Resistor_SMD:R_0402_1005Metric, symbol Device:R
- removed R33, R35: 10k, Resistor_SMD:R_0603_1608Metric, symbol Device:R
- removed R8, R9: 0, Resistor_SMD:R_0402_1005Metric, symbol Device:R
- removed U1, U2, U4, U5: PE42424A-Z, Snapeda:DFN6_1P5X1P5-0P5_PSM, symbol Snapeda:PE42424A-Z
- added C44: 0.1uF, Capacitor_SMD:C_0402_1005Metric, symbol Device:C
- added R14, R15, R18: 100, Resistor_SMD:R_0402_1005Metric, symbol Device:R
- C3: renamed from C6; footprint Capacitor_SMD:C_0603_1608Metric -> Capacitor_SMD:C_0402_1005Metric
- R1, R3: footprint Resistor_SMD:R_0603_1608Metric -> Resistor_SMD:R_0402_1005Metric
- R17: value 49.9 -> 100; Tolerance +/-1% -> (none)
- R23, R24: value 18 -> 68
- renumbered C4 to C1, C3 to C10, C15 to C11, C23 to C12, C28 to C13, C29 to C14, C30 to C15, C31 to C16, C39 to C17, C40 to C18, C41 to C19, C5 to C2, C42 to C20, C43 to C21, C35 to C22, C36 to C23, C37 to C24, C38 to C25, C49 to C26, C44 to C27, C45 to C28, C46 to C29, C47 to C30, C48 to C31, C50 to C32, C51 to C33, C52 to C34, C53 to C35, C54 to C36, C55 to C37, C56 to C38, C57 to C39, C7 to C4, C58 to C40, C60 to C41, C59 to C42, C61 to C43, C62 to C45, C63 to C46, C8 to C5, C9 to C6, C10 to C7, C1 to C8, C2 to C9, R12 to R10, R13 to R11, R14 to R12, R15 to R13, R18 to R16, R34 to R33, R11 to R6, R6 to R7, R7 to R8, R10 to R9, U3 to U1, U6 to U2
Connections:
- net FIL_SW_IN is gone; now on net GND: J5.3 (Pin_3)
- net FIL_SW_OUT is gone; now on net INT_OSC_ENABLE: J5.2 (Pin_2)
- net GND: now also J5.8 (Pin_8), R14.2, R15.2, R18.2
- net INT_OSC_ENABLE: no longer J5.4 (Pin_4)
- net RFOUT_B: now also C12.1
- net VCC: now also C29.1, C30.1, U2.15 (VCCMASH), U2.7 (VCCDIG)
- net at R31.2: now also J5.6 (Pin_6); no longer J5.7 (Pin_7)
- net at R30.2: now also J5.7 (Pin_7); no longer J5.8 (Pin_8)
- net at R33.2: now also J5.4 (Pin_4); no longer J5.5 (Pin_5)
- net at R32.2: now also J5.5 (Pin_5); no longer J5.6 (Pin_6)
- net at J4.1 (In): now also C44.1; no longer R24.1
- net at C26.2: now also R14.1, R15.1
- net at C7.1: now also C10.1, L2.2
- net at C6.2: now also C8.1, L1.1
- net at C32.2, R17.1: now also R18.1
- new net: C44.2, R24.1
Other:
- note added: "Dropping 0 ohm on VCCMASH and VCCDIG because routing made it hard, and they likely wont help much if changed to ferride bead anyways"
- note added: "Output A LP Filter, 5th order Chebychev, 950 MHz cutoff"
- note removed: "Output A Switched Filter Bank of 5th order Chebychev Lowpass filters: Upper path: 1050 MHz cutoff Lower path: 3000 MHz cutoff"
- note removed: "Output B Switched Filter Bank of 5th order Chebychev Lowpass filters: Upper path: 1050 MHz cutoff Lower path: 3000 MHz cutoff"
- note removed: "Since the LMX2582 only cannot output arbitrary frequencies independently on port A and B, I've decided that they will always output the same frequency (simplifies design). Therefore, the filter bank selection signal will be shared between port A and B, simplifying interface. Note: SW_IN and SW_OUT have to be logically inverted for the design to work. It was deemed that it was simpler to just addr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"
- moved on the sheet: C1, C10, C11, C12, C13, C14, C15, C16, C17, C18, C19, C2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

Commit message: vias vias all i can think about is vias
Connections:
- net RFOUT_A_F2: now reaches C9.1, L1.2, L2.1
- net RFOUT_A_TERM_F1: now reaches C26.2, R14.1, R15.1
- net RFOUT_B_SMA: now reaches C12.2, J3.1 (In)
- net RFOUT_A_SMA: now reaches C7.2, J2.1 (In)
- net RFOUT_B_TERM_F1: now reaches C32.2, R17.1, R18.1
- net RFOUT_A_F1: now reaches C6.2, C8.1, L1.1
- net RFOUT_A_F3: now reaches C10.1, C7.1, L2.2
Other:
- moved on the sheet: C12, C26, C32, C7, J3
