File: LO_PCB/LO_PCB.kicad_pcb (KiCad board)
At the start: 2 copper layers, 122 parts, among them J1 PWR, J2 LO_OUT_A, J3 LO_OUT_B, J4 OSCinP, J5 OSCinM, J6 Conn_01x08, Q1 AO3401A, U1 PE42424A-Z, U2 PE42424A-Z, U3 TPS7A9101DSKT, U4 PE42424A-Z, U5 PE42424A-Z, U6 LMX2582RHAR

Commit message: started on layout
Parts:
- removed the C43 at (55.0, 73.3)
- removed the C45 at (55.0, 75.8)
- removed the C48 at (55.0, 78.3)
- removed the J5 at (52.9, 51.3)
- removed the R26 at (95.0, 48.5)
- added C41: 10nF, Capacitor_SMD:C_0402_1005Metric, F.Cu at (114.2, 88.4)
- added C42: 100pF, Capacitor_SMD:C_0402_1005Metric, F.Cu at (114.2, 91.3)
- moved J3 133.7 mm to (188.1, 115.5), turned to 0 degrees
- moved C50 129.9 mm to (210.3, 101.0)
- moved C49 129.4 mm to (210.3, 97.0)
- moved R15 127.6 mm to (205.5, 108.8)
- moved R14 126.7 mm to (205.5, 104.8)
- moved R13 125.7 mm to (205.5, 100.6)
- moved R12 124.8 mm to (205.5, 96.6)
- moved R6 124.5 mm to (201.3, 100.6)
- moved C10 112.8 mm to (185.0, 93.9)
- moved J2 112.5 mm to (187.8, 82.5)
- moved C23 111.9 mm to (184.9, 107.1)
- moved C26 110.0 mm to (182.5, 104.4)
- moved L8 109.8 mm to (177.6, 109.6), turned to -90 degrees
- moved C27 109.7 mm to (182.5, 105.4)
- moved C13 109.0 mm to (182.7, 91.2)
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- renumbered C40 to C39, C41 to C40, C39 to C43, C42 to C44, C44 to C45, C49 to C48, C50 to C49, C51 to C50, C52 to C51, C53 to C52, C54 to C53, C55 to C54, C56 to C55, C57 to C56, C58 to C57, C59 to C58, C60 to C59, C61 to C60, C62 to C61, C63 to C62, C64 to C63, J6 to J5, R27 to R26, R28 to R27, R29 to R28, R30 to R29, R31 to R30, R32 to R31, R33 to R32, R34 to R33, R35 to R34, R36 to R35
Connections:
- net /RF_FIL_SW_IN renamed /FIL_SW_IN
- net /RF_FIL_SW_OUT renamed /FIL_SW_OUT
Other:
- board outline added: 60.8 x 34.4 mm
- copper layers 2 -> 4

Commit message: initial placement done, todo: CPWG and all the other routing
Parts:
- removed the C11 at (170.4, 95.5)
- removed the C12 at (170.4, 96.5)
- removed the C13 at (182.7, 91.2)
- removed the C14 at (182.7, 92.3)
- removed the C16 at (174.6, 96.4)
- removed the C17 at (176.6, 97.5)
- removed the C18 at (178.7, 97.4)
- removed the C19 at (174.2, 104.9)
- removed the C20 at (177.2, 103.9)
- removed the C21 at (179.2, 104.9)
- removed the C22 at (168.0, 107.2)
- removed the C24 at (170.2, 108.8)
- removed the C25 at (170.2, 109.9)
- removed the C26 at (182.5, 104.4)
- removed the C27 at (182.5, 105.4)
- removed the C32 at (174.6, 109.5)
- removed the C33 at (176.6, 110.5)
- removed the C34 at (178.6, 110.5)
- removed L3, L4, L7, L8: 3.9nH, Inductor_SMD:L_0402_1005Metric
- removed L5, L6: 11nH, Inductor_SMD:L_0402_1005Metric
- removed the R16 at (114.1, 105.4)
- removed the R33 at (101.4, 98.0)
- removed R35: 10k, Resistor_SMD:R_0603_1608Metric
- removed the R8 at (109.9, 101.4)
- removed the R9 at (109.9, 105.4)
- removed the U1 at (170.6, 93.8)
- removed the U2 at (182.5, 93.9)
- removed U4, U5: PE42424A-Z, Snapeda:DFN6_1P5X1P5-0P5_PSM
- added C44: 0.1uF, Capacitor_SMD:C_0402_1005Metric, F.Cu at (141.8, 99.5)
- added R14: 100, Resistor_SMD:R_0402_1005Metric, F.Cu at (167.4, 103.3)
- added R15: 100, Resistor_SMD:R_0402_1005Metric, F.Cu at (168.4, 102.2)
- added R18: 100, Resistor_SMD:R_0402_1005Metric, F.Cu at (159.9, 109.4)
- C3: renamed from C6; footprint Capacitor_SMD:C_0603_1608Metric -> Capacitor_SMD:C_0402_1005Metric
- R1, R3: footprint Resistor_SMD:R_0603_1608Metric -> Resistor_SMD:R_0402_1005Metric
- R17: value 49.9 -> 100
- R23, R24: value 18 -> 68
- moved C15 90.7 mm to (170.3, 80.8), turned to 90 degrees
- moved C14 86.9 mm to (168.2, 80.8), turned to 90 degrees
- moved C13 83.9 mm to (166.6, 80.8), turned to 90 degrees
- moved C16 82.7 mm to (171.9, 80.8), turned to 90 degrees
- moved C22 79.4 mm to (168.6, 84.8)
- moved C25 79.2 mm to (168.5, 90.0)
- moved C23 79.2 mm to (168.6, 86.4)
- moved C24 79.2 mm to (168.6, 88.4)
- moved C4 77.1 mm to (162.4, 84.7), turned to -90 degrees
- moved C3 76.2 mm to (161.6, 82.2), turned to 90 degrees
- moved C5 75.9 mm to (160.8, 84.7), turned to -90 degrees
- moved C11 71.7 mm to (155.0, 81.0), turned to 90 degrees
- moved C1 71.3 mm to (156.1, 84.1), turned to -90 degrees
- moved C2 69.2 mm to (154.4, 84.1), turned to -90 degrees
- moved R5 68.5 mm to (165.4, 84.8)
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- renumbered C4 to C1, C3 to C10, C15 to C11, C23 to C12, C28 to C13, C29 to C14, C30 to C15, C31 to C16, C39 to C17, C40 to C18, C41 to C19, C5 to C2, C42 to C20, C43 to C21, C35 to C22, C36 to C23, C37 to C24, C38 to C25, C49 to C26, C44 to C27, C45 to C28, C46 to C29, C47 to C30, C48 to C31, C50 to C32, C51 to C33, C52 to C34, C53 to C35, C54 to C36, C55 to C37, C56 to C38, C57 to C39, C7 to C4, C58 to C40, C60 to C41, C59 to C42, C61 to C43, C62 to C45, C63 to C46, C8 to C5, C9 to C6, C10 to C7, C1 to C8, C2 to C9, R12 to R10, R13 to R11, R14 to R12, R15 to R13, R18 to R16, R34 to R33, R11 to R6, R6 to R7, R7 to R8, R10 to R9, U3 to U1, U6 to U2
Connections:
- C10 pad 1: Net-(U2-RF2) -> Net-(C10-Pad1)
- C12 pad 1: Net-(U5-RFC) -> /RFOUT_B
- C29 pad 1: Net-(U6-VCCDIG) -> VCC
- C30 pad 1: Net-(U6-VCCMASH) -> VCC
- C6 pad 2: Net-(U1-RFC) -> Net-(C6-Pad2)
- C7 pad 1: Net-(U2-RFC) -> Net-(C10-Pad1)
- C8 pad 1: Net-(U1-RF1) -> Net-(C6-Pad2)
- J5 pad 2: /FIL_SW_OUT -> /INT_OSC_ENABLE
- J5 pad 3: /FIL_SW_IN -> GND
- J5 pad 4: /INT_OSC_ENABLE -> Net-(J5-Pin_4)
- J5 pad 8: Net-(J5-Pin_8) -> GND
- L1 pad 1: Net-(U1-RF1) -> Net-(C6-Pad2)
- L2 pad 2: Net-(U2-RF2) -> Net-(C10-Pad1)
- R24 pad 1: Net-(J4-In) -> Net-(C44-Pad2)
- R30 pad 2: Net-(J5-Pin_8) -> Net-(J5-Pin_7)
- R31 pad 2: Net-(J5-Pin_7) -> Net-(J5-Pin_6)
- R32 pad 2: Net-(J5-Pin_6) -> Net-(J5-Pin_5)
- R33 pad 2: Net-(J5-Pin_5) -> Net-(J5-Pin_4)
- U1 pad V: (no net) -> GND
- U2 pad 15: Net-(U6-VCCMASH) -> VCC
- U2 pad 7: Net-(U6-VCCDIG) -> VCC
- U2 pad V: (no net) -> GND
Routing:
- added copper zone on F.Cu, net GND
- added copper zone on In1.Cu, net GND
- added copper zone on In2.Cu, net GND
Other:
- board size 60.8 x 34.4 mm -> 50 x 42.5 mm

Commit message: vias vias all i can think about is vias
Parts:
- moved R27 2.17 mm to (145.1, 100.0)
- moved R23 1.14 mm to (146.2, 99.0)
- moved R24 0.45 mm to (143.5, 99.5)
- moved C44 0.29 mm to (141.5, 99.5)
- moved C29 0.18 mm to (153.3, 98.3)
- moved C40 0.18 mm to (152.2, 96.6)
- moved R19 0.18 mm to (152.2, 95.0)
- moved R15 0.13 mm to (168.4, 102.3)
- moved R10 0.06 mm to (158.1, 104.5)
- moved R11 0.06 mm to (160.1, 104.5)
- moved R18 0.06 mm to (159.9, 109.4)
- moved C17 0.05 mm to (160.1, 106.5)
Connections:
- net Net-(C10-Pad1) renamed /RFOUT_A_F3
- net Net-(C26-Pad2) renamed /RFOUT_A_TERM_F1
- net Net-(C32-Pad2) renamed /RFOUT_B_TERM_F1
- net Net-(C6-Pad2) renamed /RFOUT_A_F1
- net Net-(C9-Pad1) renamed /RFOUT_A_F2
- net Net-(J2-In) renamed /RFOUT_A_SMA
- net Net-(J3-In) renamed /RFOUT_B_SMA
- U1 pad V: GND -> (no net)
- U2 pad V: GND -> (no net)
Routing:
- net /RFOUT_B: track 0.00 -> 22.2 mm
- net /RFOUT_A: track 0.00 -> 9.32 mm
- net VccRF: track 0.00 -> 7.14 mm
- net /RFOUT_B_TERM: track 0.00 -> 6.94 mm
- net /RFOUT_B_SMA: track 0.00 -> 5.49 mm
- net /RFOUT_A_SMA: track 0.00 -> 5.43 mm
- net /RFOUT_A_TERM: track 0.00 -> 5.30 mm
- net Net-(U2-OSCINP): track 0.00 -> 4.39 mm
- net Net-(U2-OSCINM): track 0.00 -> 4.39 mm
- net Net-(R23-Pad2): track 0.00 -> 3.27 mm
- net /RFOUT_A_TERM_F1: track 0.00 -> 2.72 mm
- net /RFOUT_A_F3: track 0.00 -> 2.51 mm
- net /RFOUT_A_F1: track 0.00 -> 2.39 mm
- net /RFOUT_A_F2: track 0.00 -> 2.13 mm
- net /RFOUT_B_TERM_F1: track 0.00 -> 1.95 mm
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
Commit message: LO board v1 layout finished
Parts:
- moved R29 3.46 mm to (155.8, 111.8), turned to 90 degrees
- moved R7 1.16 mm to (154.0, 90.9)
- moved R30 1.11 mm to (157.7, 114.2), turned to 180 degrees
- moved R19 1.10 mm to (151.8, 94.1), turned to 135 degrees
- moved R20 0.96 mm to (152.7, 109.5), turned to 180 degrees
- moved C34 0.93 mm to (157.8, 92.6)
- moved C36 0.93 mm to (156.3, 92.6)
- moved C43 0.93 mm to (159.3, 92.6)
- moved C38 0.90 mm to (152.8, 93.0)
- moved C40 0.88 mm to (151.4, 96.3)
- moved C37 0.84 mm to (155.3, 105.6)
- moved R9 0.70 mm to (152.5, 103.2)
- moved C27 0.69 mm to (154.4, 92.8)
- moved C35 0.53 mm to (153.5, 107.0)
- moved C28 0.51 mm to (164.6, 95.7)
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Connections:
- R30 pad 1: Net-(U2-CSB) -> Net-(U2-MUXOUT)
- R31 pad 1: Net-(U2-SDI) -> Net-(U2-CSB)
- R32 pad 1: Net-(U2-SCK) -> Net-(U2-SDI)
- R33 pad 1: Net-(U2-MUXOUT) -> Net-(U2-SCK)
- U1 pad 5: unconnected-(U1-PG-Pad5) -> GND
Routing:
- net VCC: track 0.00 -> 91.1 mm, vias 0 -> 3
- net VccRF: track 7.14 -> 56.3 mm, vias 0 -> 4
- net /INT_OSC_ENABLE: track 0.00 -> 30.8 mm, vias 0 -> 2
- net Net-(U2-CSB): track 0.00 -> 22.5 mm, vias 0 -> 2
- net Net-(U2-VTUNE): track 0.00 -> 17.7 mm, vias 0 -> 2
- net Net-(U2-SCK): track 0.00 -> 16.9 mm, vias 0 -> 2
- net Net-(U2-SDI): track 0.00 -> 16.7 mm, vias 0 -> 2
- net Net-(U2-MUXOUT): track 0.00 -> 15.7 mm, vias 0 -> 2
- net Net-(U2-CPOUT): track 0.00 -> 8.16 mm
- net Net-(U2-VCCVCO2): track 0.00 -> 6.81 mm
- net Net-(U2-VCCVCO): track 0.00 -> 5.83 mm
- net Net-(J4-In): track 0.00 -> 5.37 mm
- net Net-(Q1-S): track 0.00 -> 5.08 mm, vias 0 -> 2
- net Net-(J1-Pin_2): track 0.00 -> 4.60 mm
- net Net-(XTAL1-VCC): track 0.00 -> 4.05 mm
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- added copper zone on F.Cu, net +3V3
- added copper zone on F.Cu, net Net-(Q1-S)
- added copper zone on F.Cu, net VCC
- added copper zone on F.Cu, net VccRF
Other:
- board text added: "+"
- board text added: "-"

Commit message: stuff and added nice border
Parts:
- removed J5: Conn_01x08, Connector_PinHeader_2.54mm:PinHeader_1x08_P2.54mm_Vertical
- added C44: 10uF, Capacitor_SMD:C_0603_1608Metric, F.Cu at (146.9, 88.4)
- added H1: MountingHole_Pad, MountingHole:MountingHole_2.2mm_M2_Pad_Via, F.Cu at (138.8, 80.5)
- added H2: MountingHole_Pad, MountingHole:MountingHole_2.2mm_M2_Pad_Via, F.Cu at (138.8, 117.0)
- added H3: MountingHole_Pad, MountingHole:MountingHole_2.2mm_M2_Pad_Via, F.Cu at (181.2, 80.5)
- added H4: MountingHole_Pad, MountingHole:MountingHole_2.2mm_M2_Pad_Via, F.Cu at (181.2, 117.0)
- added J2: Conn_01x06, Connector_PinHeader_2.54mm:PinHeader_1x06_P2.54mm_Vertical, F.Cu at (146.7, 116.8)
- C43: renamed from C42; value 1uF -> 0.1uF
- R22: value 10 -> 1
- R23: value 68 -> 47
- R24: value 68 -> 18
- moved C43 2.85 mm to (143.8, 88.4), turned to 180 degrees
- moved J1 1.23 mm to (143.9, 82.7)
- moved C21 0.10 mm to (161.3, 102.3)
- moved C40 0.10 mm to (151.3, 96.3)
- renumbered C43 to C42, C44 to C45, C45 to C46, C46 to C47, J2 to LO_OUT_A, J3 to LO_OUT_B, J4 to OSCIn
Routing:
- net Net-(U2-CSB): track 22.5 -> 25.2 mm
- net Net-(XTAL1-VCC): track 4.05 -> 5.53 mm
- net Net-(J1-Pin_2): track 4.60 -> 3.38 mm
- net Net-(U2-MUXOUT): track 15.7 -> 16.8 mm
- net /INT_OSC_ENABLE: track 30.8 -> 31.8 mm
- net Net-(U2-SCK): track 16.9 -> 17.7 mm
- net VCC: track 91.1 -> 91.8 mm, vias 3 -> 4
- net GND: vias 275 -> 350
- added copper zone on B.Cu, net GND
Other:
- board size 50 x 42.5 mm -> 50 x 44 mm
