File: LO_PCB/LO_PCB.kicad_pcb (KiCad board)
At the start: 4 copper layers, 50 x 44 mm, 99 parts, among them J1 PWR, J2 Conn_01x06, Q1 AO3401A, U1 TPS7A9101DSKT, U2 LMX2582RHAR, X1 TB612-100.0M

Commit message: updated the symbol in LO board from lmx2582 to lmx2592 in order to cover the upper range of the 5Ghz spectrum. drop in replacement
Parts:
- C47, C48, C49: value 1nF -> 10nF
- U2: value LMX2582RHAR -> LMX2592RHAR
Changed lines of the file:
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@@
 			)
 		)
-		(property "Value" "1nF"
+		(property "Value" "10nF"
 			(at 0.065 1.235 0)
 			(layer "F.Fab")
@@
 			)
 		)
-		(property "Dielectric" "C0G/NP0"
+		(property "Dielectric" "X7R"
 			(at 0 0 0)
 			(unlocked yes)
@@
 			)
 		)
-		(property "Tolerance" "+/-5%"
+		(property "Tolerance" "+/-10%"
 			(at 0 0 0)
 			(unlocked yes)
@@
 			)
 		)
-		(property "MPN" "GRM1555C1H102JA01D"
+		(property "MPN" "GRM155R71H103KA88D"
 			(at 0 0 0)
 			(unlocked yes)
@@
 			)
 		)
-		(property "Value" "1nF"
+		(property "Value" "10nF"
 			(at 0 1.16 0)
 			(layer "F.Fab")
@@
 			)
 		)
-		(property "Dielectric" "C0G/NP0"
+		(property "Dielectric" "X7R"
 			(at 0 0 0)
 			(unlocked yes)
@@
 			)
 		)
-		(property "Tolerance" "+/-5%"
+		(property "Tolerance" "+/-10%"
 			(at 0 0 0)
 			(unlocked yes)
@@
 			)
 		)
-		(property "MPN" "GRM1555C1H102JA01D"
+		(property "MPN" "GRM155R71H103KA88D"
 			(at 0 0 0)
 			(unlocked yes)
@@
 		(layer "F.Cu")
 		(at 157.556801 98.4888)
-		(tags "LMX2582RHAR ")
+		(tags "LMX2592RHAR ")
 		(property "Reference" "U2"
 			(at 0 0 0)
@@
 			)
 		)
-		(property "Value" "LMX2582RHAR"
+		(property "Value" "LMX2592RHAR"
 			(at 0 0 0)
 			(unlocked yes)
@@
 			)
 		)
-		(property "Datasheet" "https://www.ti.com/lit/gpn/lmx2582"
+		(property "Datasheet" "https://www.ti.com/lit/gpn/lmx2592"
 			(at 0 0 0)
 			(layer "F.Fab")
@@
 			)
 		)
-		(property "MPN" "LMX2582RHAR"
+		(property "MPN" "LMX2592RHAR"
 			(at 0 0 0)
 			(unlocked yes)
@@
 			)
 		)
-		(property "Value" "1nF"
+		(property "Value" "10nF"
 			(at 0 1.16 0)
 			(layer "F.Fab")
@@
 			)
 		)
-		(property "Dielectric" "C0G/NP0"
+		(property "Dielectric" "X7R"
 			(at 0 0 0)
 			(unlocked yes)
@@
 			)
 		)
-		(property "Tolerance" "+/-5%"
+		(property "Tolerance" "+/-10%"
 			(at 0 0 0)
 			(unlocked yes)
@@
 			)
 		)
-		(property "MPN" "GRM1555C1H102JA01D"
+		(property "MPN" "GRM155R71H103KA88D"
 			(at 0 0 0)
 			(unlocked yes)
